File: Schematic/PSU/PSU.sch (KiCad schematic (older format))
At the start: 36 parts, among them J1 Trafo sec 26V, J2 Trafo pri 230V, J3 230V input, J4 Power switch, J5 To timer, J6 UV_Panel_1, J7 UV_Panel_2, Q1 2N7000, Q2 2N7000, U1 LM338, U2 MC7805CT-BP

Commit message: PSU board: Added temperature sensor and fan driver. 12V relays.
Parts:
- removed C5: 1µF, Capacitor_THT:C_Rect_L18.0mm_W8.0mm_P15.00mm_FKS3_FKP3, symbol Device:C
- added C10, C8: 100nF, Capacitor_THT:C_Rect_L7.2mm_W2.5mm_P5.00mm_FKS2_FKP2_MKS2_MKP2, symbol Device:C
- added C5, C7, C9: 10µF, Capacitor_THT:CP_Radial_D5.0mm_P2.00mm, symbol Device:CP
- added J7: Timer I/O, myDevices:KF2510-4P, symbol Connector_Generic:Conn_01x04
- added J9: 12V FAN, myDevices:KF2510-2P, symbol Connector_Generic:Conn_01x02
- added Q3: 2N7000, digikey-footprints:TO-92-3, symbol dk_Transistors-FETs-MOSFETs-Single:2N7000
- added R4: 4.7kΩ, Resistor_THT:R_Axial_DIN0207_L6.3mm_D2.5mm_P7.62mm_Horizontal, symbol Device:R
- added R7: 10kΩ, Resistor_THT:R_Axial_DIN0207_L6.3mm_D2.5mm_P7.62mm_Horizontal, symbol Device:R
- added U2: DS18B20+, TO127P482X368X883-3, symbol IFS-Sensors:DS18B20+
- added U3: LM7812_TO220, digikey-footprints:TO-220-3, symbol Regulator_Linear:LM7812_TO220
- C4, C6: value 1µF -> 100nF; footprint Capacitor_THT:C_Rect_L18.0mm_W8.0mm_P15.00mm_FKS3_FKP3 -> Capacitor_THT:C_Rect_L7.2mm_W2.5mm_P5.00mm_FKS2_FKP2_MKS2_MKP2
- J8: renamed from J5; value To timer -> Timer power; footprint myDevices:KF2510-4P -> myDevices:KF2510-2P; symbol Connector_Generic:Conn_01x04 -> Connector_Generic:Conn_01x02
- RLY1, RLY2: value G5LE-14_DC36 -> G5LE-14_DC12
- renumbered C2 to C1, C1 to C2, F2 to F1, F1 to F2, J6 to J5, J7 to J6, R5 to R1, R1 to R2, R2 to R3, R3 to R5, R4 to R6, U2 to U4
Connections:
- net +5V: now also C10.1, C9.1, R4.1, U2.3 (VDD); no longer C6.1
- net GND: now also J8.2 (Pin_2), C10.2, C5.2, C7.2, C8.2, C9.2, Q3.1 (S), R7.2, U2.1 (GND), U3.2 (GND); no longer J8.4 (Pin_4)
- net VCC: now also C6.1, C5.1, U3.1 (VI); no longer U4.1 (IN)
- net at Q1.2 (G), R3.1: now also J7.2 (Pin_2); no longer J8.3 (Pin_3)
- net at Q2.2 (G), R5.1: now also J7.1 (Pin_1); no longer J8.2 (Pin_2)
- net +36V: no longer names the net of C1.1, C3.1, C4.1, D1.1 (+), U1.3 (IN)
- net +36V: no longer D2.1 (K), D3.1 (K), RLY1.2 (COIL), RLY2.2 (COIL)
- new net: J7.3 (Pin_3), R4.2, U2.2 (DQ)
- new net: J7.4 (Pin_4), Q3.2 (G), R7.1
- new net: J9.1 (Pin_1), Q3.3 (D)
- new net +12V: C7.1, C8.1, D2.1 (K), D3.1 (K), J9.2 (Pin_2), RLY1.2 (COIL), RLY2.2 (COIL), U3.3 (VO), U4.1 (IN)
Other:
- moved on the sheet: D2, D3, D4, J5, J6, Q1, Q2, R3, R5, R6, RLY1, RLY2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
