File: Schematic/PSU/PSU.kicad_pcb (KiCad board)
At the start: 2 copper layers, 100 x 76.5 mm, 36 parts, among them J1 Trafo sec 26V, J2 Trafo pri 230V, J3 230V input, J4 Power switch, J5 To timer, J6 UV_Panel_1, J7 UV_Panel_2, Q1 2N7000, Q2 2N7000, U1 LM338, U2 MC7805CT-BP

Commit message: PSU board: Added temperature sensor and fan driver. 12V relays.
Parts:
- removed the R1 at (111.0, 44.0)
- added C10: 100nF, Capacitor_THT:C_Rect_L7.2mm_W2.5mm_P5.00mm_FKS2_FKP2_MKS2_MKP2, F.Cu at (101.0, 46.0)
- added C7: 10µF, Capacitor_THT:CP_Radial_D5.0mm_P2.00mm, F.Cu at (111.5, 51.8)
- added C8: 100nF, Capacitor_THT:C_Rect_L7.2mm_W2.5mm_P5.00mm_FKS2_FKP2_MKS2_MKP2, F.Cu at (110.8, 46.0)
- added C9: 10µF, Capacitor_THT:CP_Radial_D5.0mm_P2.00mm, F.Cu at (103.2, 51.8)
- added J7: Timer I/O, myDevices:KF2510-4P, F.Cu at (194.2, 59.0)
- added J9: 12V FAN, myDevices:KF2510-2P, F.Cu at (104.0, 59.4)
- added Q3: 2N7000, digikey-footprints:TO-92-3, F.Cu at (106.6, 65.0)
- added R2: 240Ω, Resistor_THT:R_Axial_DIN0207_L6.3mm_D2.5mm_P7.62mm_Horizontal, F.Cu at (132.2, 41.8)
- added R4: 4.7kΩ, Resistor_THT:R_Axial_DIN0207_L6.3mm_D2.5mm_P7.62mm_Horizontal, F.Cu at (185.2, 45.5)
- added R7: 10kΩ, Resistor_THT:R_Axial_DIN0207_L6.3mm_D2.5mm_P7.62mm_Horizontal, F.Cu at (113.6, 66.4)
- added U2: DS18B20+, IFS-IC:TO127P482X368X883-3, F.Cu at (159.2, 39.0)
- added U3: LM7812_TO220, digikey-footprints:TO-220-3, F.Cu at (120.5, 39.5)
- C4, C6: value 1µF -> 100nF; footprint Capacitor_THT:C_Rect_L18.0mm_W8.0mm_P15.00mm_FKS3_FKP3 -> Capacitor_THT:C_Rect_L7.2mm_W2.5mm_P5.00mm_FKS2_FKP2_MKS2_MKP2
- C5: value 1µF -> 10µF; footprint Capacitor_THT:C_Rect_L18.0mm_W8.0mm_P15.00mm_FKS3_FKP3 -> Capacitor_THT:CP_Radial_D5.0mm_P2.00mm
- J8: renamed from J5; value To timer -> Timer power; footprint myDevices:KF2510-4P -> myDevices:KF2510-2P
- RLY1, RLY2: value G5LE-14_DC36 -> G5LE-14_DC12
- moved C4 29.6 mm to (151.5, 46.0), turned to 180 degrees
- moved U1 24.9 mm to (146.4, 39.5)
- moved C5 16.2 mm to (119.8, 51.8)
- moved J8 9.22 mm to (194.2, 50.5), turned to 270 degrees
- moved C6 7.76 mm to (120.5, 46.0), turned to 0 degrees
- moved C1 4.00 mm to (135.5, 50.5)
- renumbered C2 to C1, C1 to C2, F2 to F1, F1 to F2, J6 to J5, J7 to J6, R5 to R1, R2 to R3, R3 to R5, R4 to R6, U2 to U4
Connections:
- C1 pad 1: +36V -> Net-(C1-Pad1)
- C3 pad 1: +36V -> Net-(C1-Pad1)
- C4 pad 1: +36V -> Net-(C1-Pad1)
- C6 pad 1: +5V -> VCC
- D1 pad 1: +36V -> Net-(C1-Pad1)
- D2 pad 1: +36V -> +12V
- D3 pad 1: +36V -> +12V
- J8 pad 2: Net-(J5-Pad2) -> GND
- Q1 pad 2: Net-(J5-Pad3) -> Net-(J7-Pad2)
- Q2 pad 2: Net-(J5-Pad2) -> Net-(J7-Pad1)
- R3 pad 1: Net-(J5-Pad3) -> Net-(J7-Pad2)
- R5 pad 1: Net-(J5-Pad2) -> Net-(J7-Pad1)
- RLY1 pad 2: +36V -> +12V
- RLY2 pad 2: +36V -> +12V
- U1 pad 3: +36V -> Net-(C1-Pad1)
- U4 pad 1: VCC -> +12V
Routing:
- net Net-(J7-Pad4): track 0.00 -> 173.0 mm
- net +12V: track 0.00 -> 165.6 mm
- net +36V: track 146.0 -> 0.00 mm
- net Net-(J7-Pad3): track 0.00 -> 55.7 mm
- net Net-(C1-Pad1): track 0.00 -> 53.1 mm
- net Net-(J7-Pad2): track 0.00 -> 28.3 mm
- net Net-(J5-Pad3): track 25.4 -> 0.00 mm
- net +5V: track 131.9 -> 156.0 mm
- net Net-(J7-Pad1): track 0.00 -> 23.0 mm
- net Net-(J5-Pad2): track 15.5 -> 0.00 mm
- net GND: track 0.00 -> 8.24 mm, vias 0 -> 32
- net Net-(J9-Pad1): track 0.00 -> 4.35 mm
- net Net-(R2-Pad2): track 51.9 -> 48.9 mm
- net VCC: track 120.4 -> 119.3 mm
- added copper zone on F.Cu, net GND
Other:
- board text added: "+"
- board text added: "-"
- board text added: "FAN 12V"
- board text added: "FanCtrl"
- board text added: "RelayCtrl1"
- board text added: "RelayCtrl2"
- board text added: "Sens"
- board text removed: "Ctrl1"
- board text removed: "Ctrl2"

Commit message: PSU: corrected silkscreen for timer inputs
Routing:
- net VCC: track 119.3 -> 115.7 mm
Changed lines of the file:
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@@
     (thickness 1.6)
     (drawings 22)
-    (tracks 187)
+    (tracks 188)
     (zones 0)
     (modules 47)
@@
     (effects (font (size 1 1) (thickness 0.15)))
   )
-  (gr_text RelayCtrl1 (at 187 55.2) (layer F.SilkS)
+  (gr_text RelayCtrl2 (at 187 55.2) (layer F.SilkS)
     (effects (font (size 1 1) (thickness 0.15)))
   )
-  (gr_text RelayCtrl2 (at 187 57.8) (layer F.SilkS)
+  (gr_text RelayCtrl1 (at 187 57.8) (layer F.SilkS)
     (effects (font (size 1 1) (thickness 0.15)))
   )
@@
   (segment (start 192.099999 79.200001) (end 179.400001 79.200001) (width 3) (layer F.Cu) (net 3))
   (segment (start 195 76.3) (end 192.099999 79.200001) (width 3) (layer F.Cu) (net 3))
-  (segment (start 174.449999 56.199997) (end 174.449999 74.249999) (width 2) (layer B.Cu) (net 3))
-  (segment (start 165.500001 47.249999) (end 174.449999 56.199997) (width 2) (layer B.Cu) (net 3))
-  (segment (start 155.719997 47.249999) (end 165.500001 47.249999) (width 2) (layer B.Cu) (net 3))
-  (segment (start 174.449999 74.249999) (end 176.5 76.3) (width 2) (layer B.Cu) (net 3))
-  (segment (start 148.96 40.490002) (end 155.719997 47.249999) (width 2) (layer B.Cu) (net 3))
   (segment (start 148.96 39.7) (end 148.96 40.490002) (width 2) (layer B.Cu) (net 3))
   (segment (start 121 41.8) (end 120.5 42.3) (width 1) (layer F.Cu) (net 3))
@@
   (segment (start 120.5 51) (end 119.75 51.75) (width 1) (layer F.Cu) (net 3))
   (segment (start 120.5 46) (end 120.5 51) (width 1) (layer F.Cu) (net 3))
+  (segment (start 150.179999 42.250001) (end 149.170001 41.240003) (width 3) (layer B.Cu) (net 3))
+  (segment (start 151.524003 42.250001) (end 150.179999 42.250001) (width 3) (layer B.Cu) (net 3))
+  (segment (start 154.050001 57.600003) (end 154.050001 44.775999) (width 3) (layer B.Cu) (net 3))
+  (segment (start 172.749998 76.3) (end 154.050001 57.600003) (width 3) (layer B.Cu) (net 3))
+  (segment (start 154.050001 44.775999) (end 151.524003 42.250001) (width 3) (layer B.Cu) (net 3))
+  (segment (start 176.5 76.3) (end 172.749998 76.3) (width 3) (layer B.Cu) (net 3))
   (segment (start 105.749999 41.250001) (end 101 46) (width 1) (layer B.Cu) (net 4))
   (segment (start 112.329999 41.250001) (end 105.749999 41.250001) (width 1) (layer B.Cu) (net 4))
