File: Schematic/Timer/Timer.sch (KiCad schematic (older format))
At the start: 39 parts, among them J1 FIRMWARE, J2 Analog header, J3 I2C Header, J4 GPIO Header, J5 MCP Header, J6 Power, SW1 Rotary_Encoder_Switch, U1 Display_OLED_0.96_I2C, U2 DS3231MZ, U3 MCP23017-E_SO, U4 ATMEGA328P-AU_Arduino, Y1 16MHz

Commit message: New timer with the more precise DS3231 + more digital I/O ports exposed.
Parts:
- removed JP1: Jumper_2_Open, Connector_PinHeader_2.54mm:PinHeader_1x02_P2.54mm_Vertical, symbol Jumper:Jumper_2_Open
- removed U2: DS3231MZ, Package_SO:SOIC-8_3.9x4.9mm_P1.27mm, symbol Timer_RTC:DS3231MZ
- added C3: 100nF, Capacitor_SMD:C_0805_2012Metric_Pad1.15x1.40mm_HandSolder, symbol Device:C
- added C9: 1µF, Capacitor_SMD:C_0805_2012Metric_Pad1.15x1.40mm_HandSolder, symbol Device:C
- added U1: DS3231M, Package_SO:SOIC-16W_7.5x10.3mm_P1.27mm, symbol Timer_RTC:DS3231M
- C2: renamed from C1; value 1µF -> 100nF
- J2: renamed from J6; value Power -> Power 3.3/5 V
- J5: renamed from J4; footprint myDevices:KF2510-5P -> myDevices:KF2510-8P; symbol Connector_Generic:Conn_01x05 -> Connector_Generic:Conn_01x08
- Y1: value 16MHz -> 8/16MHz
- renumbered C2 to C1, C3 to C4, C4 to C5, C5 to C6, C6 to C7, C7 to C8, J2 to J3, J3 to J4, J5 to J6, R3 to R1, R1 to R3, S1 to S0, S4 to S1, S5 to S3, S3 to S4, S6 to S5, U1 to U2
Connections:
- net +BATT: now also C3.1, U1.14 (VBAT)
- net BUTTON1: now also S1.2; no longer S2.2
- net BUTTON2: now also S2.2, U3.4 (11_(GPB3)); no longer S4.2, U3.3 (10_(GPB2))
- net BUTTON3: now also S3.2, U3.3 (10_(GPB2)); no longer S1.2, U3.4 (11_(GPB3))
- net BUTTON4: now also S4.2, U3.6 (13_(GPB5)); no longer S3.2, U3.5 (12_(GPB4))
- net BUTTON5: now also U3.5 (12_(GPB4)); no longer U3.6 (13_(GPB5))
- net D10: now also J5.4 (Pin_4); no longer J5.1 (Pin_1)
- net D11: now also J5.5 (Pin_5); no longer J5.2 (Pin_2)
- net D12: now also J5.6 (Pin_6); no longer J5.3 (Pin_3)
- net D13: now also J5.7 (Pin_7); no longer J5.4 (Pin_4)
- net GND: now also J5.8 (Pin_8), C3.2, C9.1, U1.10 (GND), U1.11 (GND), U1.12 (GND), U1.13 (GND), U1.5 (GND), U1.6 (GND), U1.7 (GND), U1.8 (GND), U1.9 (GND); no longer J5.5 (Pin_5)
- net SCL: now also U1.16 (SCL)
- net SDA: now also U1.15 (SDA)
- net ~RESET: now also U1.4 (~RST)
- net at U4.1 (D3(PWM)/INT1): now also SW1.A; no longer SW1.B
- net D6: now reaches U4.10 (D6(PWM))
- net D6: now also J5.2 (Pin_2)
- net at U4.11 (D7): now also D1.2 (A)
- net at U4.12 (D8): now also D2.2 (A); no longer D1.2 (A)
- net D9: now reaches U4.13 (D9(PWM))
- net D9: now also J5.3 (Pin_3); no longer D2.2 (A)
- net at U4.2 (D4): now also SW1.B; no longer SW1.A
- net D5: now reaches U4.9 (D5(PWM))
- net D5: now also J5.1 (Pin_1)
- net RTC_INT: now reaches R3.2
- net RTC_INT: now also U3.7 (14_(GPB6)), U1.3 (~INT~/SQW)
- net +5V renamed VCC
- net VCC: now also C9.2, U1.2 (VCC)
- no-connect marks 9 -> 6
Other:
- moved on the sheet: BAT1, C1, C2, C6, C7, D1, D2, J6, R1, R2, R3, R4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

Commit message: Code for hardware test
Parts:
- C2: value 100nF -> 1µF
Connections:
- net BUTTON0 renamed IOEXT_BTN0
- net BUTTON1 renamed IOEXT_BTN1
- net BUTTON2 renamed IOEXT_BTN2
- net BUTTON3 renamed IOEXT_BTN3
- net BUTTON4 renamed IOEXT_BTN4
- net BUTTON5 renamed IOEXT_BTN5
- net MCP_INT renamed MCP_INTA
Other:
- note added: "I2C Address: 0x3C"
- moved on the sheet: S1, S3, S5
